Commit message: Add IMU and 2D lidar sensors with Gazebo plugins

File: src/scout_mini_description/urdf/scout_mini.gazebo.xacro (robot description, xacro)
@@ -64,3 +64,115 @@
     </plugin>
   </gazebo>
+  <!-- ============================================================== -->
+  <!-- IMU sensor plugin                                              -->
+  <!-- Publishes /imu at 100 Hz on imu_link frame                      -->
+  <!-- ============================================================== -->
+  <gazebo reference="imu_link">
+    <sensor name="imu_sensor" type="imu">
+      <always_on>true</always_on>
+      <update_rate>100</update_rate>
+      <visualize>false</visualize>
+      <topic>__default_topic__</topic>
+      <plugin filename="libgazebo_ros_imu_sensor.so" name="imu_plugin">
+        <ros>
+          <namespace>/</namespace>
+          <remapping>~/out:=imu</remapping>
+        </ros>
+        <initial_orientation_as_reference>false</initial_orientation_as_reference>
+        <frame_name>imu_link</frame_name>
+      </plugin>
+      <imu>
+        <angular_velocity>
+          <x>
+            <noise type="gaussian">
+              <mean>0.0</mean>
+              <stddev>2e-4</stddev>
+              <bias_mean>0.0000075</bias_mean>
+              <bias_stddev>0.0000008</bias_stddev>
+            </noise>
+          </x>
+          <y>
+            <noise type="gaussian">
+              <mean>0.0</mean>
+              <stddev>2e-4</stddev>
+              <bias_mean>0.0000075</bias_mean>
+              <bias_stddev>0.0000008</bias_stddev>
+            </noise>
+          </y>
+          <z>
+            <noise type="gaussian">
+              <mean>0.0</mean>
+              <stddev>2e-4</stddev>
+              <bias_mean>0.0000075</bias_mean>
+              <bias_stddev>0.0000008</bias_stddev>
+            </noise>
+          </z>
+        </angular_velocity>
+        <linear_acceleration>
+          <x>
+            <noise type="gaussian">
+              <mean>0.0</mean>
+              <stddev>1.7e-2</stddev>
+              <bias_mean>0.1</bias_mean>
+              <bias_stddev>0.001</bias_stddev>
+            </noise>
+          </x>
+          <y>
+            <noise type="gaussian">
+              <mean>0.0</mean>
+              <stddev>1.7e-2</stddev>
+              <bias_mean>0.1</bias_mean>
+              <bias_stddev>0.001</bias_stddev>
+            </noise>
+          </y>
+          <z>
+            <noise type="gaussian">
+              <mean>0.0</mean>
+              <stddev>1.7e-2</stddev>
+              <bias_mean>0.1</bias_mean>
+              <bias_stddev>0.001</bias_stddev>
+            </noise>
+          </z>
+        </linear_acceleration>
+      </imu>
+    </sensor>
+  </gazebo>
+  <!-- 2D Lidar plugin                                                 -->
+  <!-- Publishes /scan at 10 Hz, 360°, 0.12-12m range                  -->
+  <gazebo reference="lidar_link">
+    <sensor name="lidar_sensor" type="ray">
+      <always_on>true</always_on>
+      <update_rate>10</update_rate>
+      <visualize>true</visualize>
+      <pose>0 0 0 0 0 0</pose>
+      <ray>
+        <scan>
+          <horizontal>
+            <samples>360</samples>
+            <resolution>1</resolution>
+            <min_angle>-3.14159</min_angle>
+            <max_angle>3.14159</max_angle>
+          </horizontal>
+        </scan>
+        <range>
+          <min>0.12</min>
+          <max>12.0</max>
+          <resolution>0.015</resolution>
+        </range>
+        <noise>
+          <type>gaussian</type>
+          <mean>0.0</mean>
+          <stddev>0.01</stddev>
+        </noise>
+      </ray>
+      <plugin filename="libgazebo_ros_ray_sensor.so" name="lidar_plugin">
+        <ros>
+          <namespace>/</namespace>
+          <remapping>~/out:=scan</remapping>
+        </ros>
+        <output_type>sensor_msgs/LaserScan</output_type>
+        <frame_name>lidar_link</frame_name>
+      </plugin>
+    </sensor>
+  </gazebo>
 </robot>

File: src/scout_mini_description/urdf/scout_mini.urdf.xacro (robot description, xacro)
@@ -102,4 +102,62 @@
   <xacro:wheel prefix="rear_left"   x_offset="${-wheelbase/2}" y_offset="${ track_width/2}"/>
   <xacro:wheel prefix="rear_right"  x_offset="${-wheelbase/2}" y_offset="${-track_width/2}"/>
+  <!-- IMU sensor                                                      -->
+  <!-- Mounted on the top center of base_link                          -->
+  <link name="imu_link">
+    <visual>
+      <geometry>
+        <box size="0.04 0.04 0.02"/>
+      </geometry>
+      <material name="imu_blue">
+        <color rgba="0.0 0.3 0.8 1.0"/>
+      </material>
+    </visual>
+    <collision>
+      <geometry>
+        <box size="0.04 0.04 0.02"/>
+      </geometry>
+    </collision>
+    <inertial>
+      <mass value="0.05"/>
+      <inertia
+        ixx="1e-5" ixy="0.0" ixz="0.0"
+        iyy="1e-5" iyz="0.0"
+        izz="1e-5"/>
+    </inertial>
+  </link>
+  <joint name="imu_joint" type="fixed">
+    <parent link="base_link"/>
+    <child link="imu_link"/>
+    <origin xyz="0 0 ${base_height + 0.01}" rpy="0 0 0"/>
+  </joint>
+  <!-- 2D Lidar (LSLIDAR N10-class)                                    -->
+  <!-- Mounted on the top of base_link, forward of IMU                 -->
+  <link name="lidar_link">
+    <visual>
+      <geometry>
+        <cylinder radius="0.04" length="0.06"/>
+      </geometry>
+      <material name="lidar_dark">
+        <color rgba="0.2 0.2 0.2 1.0"/>
+      </material>
+    </visual>
+    <collision>
+      <geometry>
+        <cylinder radius="0.04" length="0.06"/>
+      </geometry>
+    </collision>
+    <inertial>
+      <mass value="0.2"/>
+      <inertia
+        ixx="2e-4" ixy="0.0" ixz="0.0"
+        iyy="2e-4" iyz="0.0"
+        izz="1e-4"/>
+    </inertial>
+  </link>
+  <joint name="lidar_joint" type="fixed">
+    <parent link="base_link"/>
+    <child link="lidar_link"/>
+    <origin xyz="0.20 0 ${base_height + 0.03}" rpy="0 0 0"/>
+  </joint>
   <xacro:include filename="$(find scout_mini_description)/urdf/scout_mini.gazebo.xacro"/>
 </robot>

Commit message: Refactor sensors into parameterized xacro macros

File: src/scout_mini_description/urdf/scout_mini.gazebo.xacro (robot description, xacro)
@@ -64,115 +64,3 @@
     </plugin>
   </gazebo>
-  <!-- ============================================================== -->
-  <!-- IMU sensor plugin                                              -->
-  <!-- Publishes /imu at 100 Hz on imu_link frame                      -->
-  <!-- ============================================================== -->
-  <gazebo reference="imu_link">
-    <sensor name="imu_sensor" type="imu">
-      <always_on>true</always_on>
-      <update_rate>100</update_rate>
-      <visualize>false</visualize>
-      <topic>__default_topic__</topic>
-      <plugin filename="libgazebo_ros_imu_sensor.so" name="imu_plugin">
-        <ros>
-          <namespace>/</namespace>
-          <remapping>~/out:=imu</remapping>
-        </ros>
-        <initial_orientation_as_reference>false</initial_orientation_as_reference>
-        <frame_name>imu_link</frame_name>
-      </plugin>
-      <imu>
-        <angular_velocity>
-          <x>
-            <noise type="gaussian">
-              <mean>0.0</mean>
-              <stddev>2e-4</stddev>
-              <bias_mean>0.0000075</bias_mean>
-              <bias_stddev>0.0000008</bias_stddev>
-            </noise>
-          </x>
-          <y>
-            <noise type="gaussian">
-              <mean>0.0</mean>
-              <stddev>2e-4</stddev>
-              <bias_mean>0.0000075</bias_mean>
-              <bias_stddev>0.0000008</bias_stddev>
-            </noise>
-          </y>
-          <z>
-            <noise type="gaussian">
-              <mean>0.0</mean>
-              <stddev>2e-4</stddev>
-              <bias_mean>0.0000075</bias_mean>
-              <bias_stddev>0.0000008</bias_stddev>
-            </noise>
-          </z>
-        </angular_velocity>
-        <linear_acceleration>
-          <x>
-            <noise type="gaussian">
-              <mean>0.0</mean>
-              <stddev>1.7e-2</stddev>
-              <bias_mean>0.1</bias_mean>
-              <bias_stddev>0.001</bias_stddev>
-            </noise>
-          </x>
-          <y>
-            <noise type="gaussian">
-              <mean>0.0</mean>
-              <stddev>1.7e-2</stddev>
-              <bias_mean>0.1</bias_mean>
-              <bias_stddev>0.001</bias_stddev>
-            </noise>
-          </y>
-          <z>
-            <noise type="gaussian">
-              <mean>0.0</mean>
-              <stddev>1.7e-2</stddev>
-              <bias_mean>0.1</bias_mean>
-              <bias_stddev>0.001</bias_stddev>
-            </noise>
-          </z>
-        </linear_acceleration>
-      </imu>
-    </sensor>
-  </gazebo>
-  <!-- 2D Lidar plugin                                                 -->
-  <!-- Publishes /scan at 10 Hz, 360°, 0.12-12m range                  -->
-  <gazebo reference="lidar_link">
-    <sensor name="lidar_sensor" type="ray">
-      <always_on>true</always_on>
-      <update_rate>10</update_rate>
-      <visualize>true</visualize>
-      <pose>0 0 0 0 0 0</pose>
-      <ray>
-        <scan>
-          <horizontal>
-            <samples>360</samples>
-            <resolution>1</resolution>
-            <min_angle>-3.14159</min_angle>
-            <max_angle>3.14159</max_angle>
-          </horizontal>
-        </scan>
-        <range>
-          <min>0.12</min>
-          <max>12.0</max>
-          <resolution>0.015</resolution>
-        </range>
-        <noise>
-          <type>gaussian</type>
-          <mean>0.0</mean>
-          <stddev>0.01</stddev>
-        </noise>
-      </ray>
-      <plugin filename="libgazebo_ros_ray_sensor.so" name="lidar_plugin">
-        <ros>
-          <namespace>/</namespace>
-          <remapping>~/out:=scan</remapping>
-        </ros>
-        <output_type>sensor_msgs/LaserScan</output_type>
-        <frame_name>lidar_link</frame_name>
-      </plugin>
-    </sensor>
-  </gazebo>
 </robot>

File: src/scout_mini_description/urdf/scout_mini.urdf.xacro (robot description, xacro)
@@ -102,62 +102,19 @@
   <xacro:wheel prefix="rear_left"   x_offset="${-wheelbase/2}" y_offset="${ track_width/2}"/>
   <xacro:wheel prefix="rear_right"  x_offset="${-wheelbase/2}" y_offset="${-track_width/2}"/>
-  <!-- IMU sensor                                                      -->
-  <!-- Mounted on the top center of base_link                          -->
-  <link name="imu_link">
-    <visual>
-      <geometry>
-        <box size="0.04 0.04 0.02"/>
-      </geometry>
-      <material name="imu_blue">
-        <color rgba="0.0 0.3 0.8 1.0"/>
-      </material>
-    </visual>
-    <collision>
-      <geometry>
-        <box size="0.04 0.04 0.02"/>
-      </geometry>
-    </collision>
-    <inertial>
-      <mass value="0.05"/>
-      <inertia
-        ixx="1e-5" ixy="0.0" ixz="0.0"
-        iyy="1e-5" iyz="0.0"
-        izz="1e-5"/>
-    </inertial>
-  </link>
-  <joint name="imu_joint" type="fixed">
-    <parent link="base_link"/>
-    <child link="imu_link"/>
-    <origin xyz="0 0 ${base_height + 0.01}" rpy="0 0 0"/>
-  </joint>
-  <!-- 2D Lidar (LSLIDAR N10-class)                                    -->
-  <!-- Mounted on the top of base_link, forward of IMU                 -->
-  <link name="lidar_link">
-    <visual>
-      <geometry>
-        <cylinder radius="0.04" length="0.06"/>
-      </geometry>
-      <material name="lidar_dark">
-        <color rgba="0.2 0.2 0.2 1.0"/>
-      </material>
-    </visual>
-    <collision>
-      <geometry>
-        <cylinder radius="0.04" length="0.06"/>
-      </geometry>
-    </collision>
-    <inertial>
-      <mass value="0.2"/>
-      <inertia
-        ixx="2e-4" ixy="0.0" ixz="0.0"
-        iyy="2e-4" iyz="0.0"
-        izz="1e-4"/>
-    </inertial>
-  </link>
-  <joint name="lidar_joint" type="fixed">
-    <parent link="base_link"/>
-    <child link="lidar_link"/>
-    <origin xyz="0.20 0 ${base_height + 0.03}" rpy="0 0 0"/>
-  </joint>
   <xacro:include filename="$(find scout_mini_description)/urdf/scout_mini.gazebo.xacro"/>
+  <!-- ============================================================== -->
+  <!-- Sensor modules                                                  -->
+  <!-- ============================================================== -->
+  <xacro:include filename="$(find scout_mini_description)/urdf/sensors/imu.xacro"/>
+  <xacro:include filename="$(find scout_mini_description)/urdf/sensors/lidar_2d.xacro"/>
+  <xacro:imu_sensor
+    name="imu"
+    parent="base_link"
+    xyz="0 0 ${base_height + 0.01}"
+    rpy="0 0 0"/>
+  <xacro:lidar_2d_sensor
+    name="lidar"
+    parent="base_link"
+    xyz="0.20 0 ${base_height + 0.03}"
+    rpy="0 0 0"/>
 </robot>
