Commit message: Refactor URDF into parameterized macro with prefix and sensor flags

File: src/scout_mini_description/urdf/scout_mini.gazebo.xacro (robot description, xacro)
@@ -1,66 +1,70 @@
 <?xml version="1.0"?>
 <robot xmlns:xacro="http://www.ros.org/wiki/xacro">
-  <!-- Gazebo material colors                                         -->
-  <gazebo reference="base_link">
-    <material>Gazebo/Yellow</material>
-  </gazebo>
-  <gazebo reference="front_left_wheel_link">
-    <material>Gazebo/Black</material>
-    <mu1>1.0</mu1>
-    <mu2>1.0</mu2>
-    <kp>1000000.0</kp>
-    <kd>100.0</kd>
-  </gazebo>
-  <gazebo reference="front_right_wheel_link">
-    <material>Gazebo/Black</material>
-    <mu1>1.0</mu1>
-    <mu2>1.0</mu2>
-    <kp>1000000.0</kp>
-    <kd>100.0</kd>
-  </gazebo>
-  <gazebo reference="rear_left_wheel_link">
-    <material>Gazebo/Black</material>
-    <mu1>1.0</mu1>
-    <mu2>1.0</mu2>
-    <kp>1000000.0</kp>
-    <kd>100.0</kd>
-  </gazebo>
-  <gazebo reference="rear_right_wheel_link">
-    <material>Gazebo/Black</material>
-    <mu1>1.0</mu1>
-    <mu2>1.0</mu2>
-    <kp>1000000.0</kp>
-    <kd>100.0</kd>
-  </gazebo>
   <!-- ============================================================== -->
-  <!-- Skid-steer drive controller                                    -->
-  <!-- Drives all four wheels from /cmd_vel, publishes /odom + TF     -->
+  <!-- Gazebo macro: per-robot material + skid-steer plugin            -->
   <!-- ============================================================== -->
-  <gazebo>
-    <plugin name="skid_steer_controller" filename="libgazebo_ros_diff_drive.so">
-      <ros>
-        <namespace>/</namespace>
-        <remapping>cmd_vel:=cmd_vel</remapping>
-        <remapping>odom:=odom</remapping>
-      </ros>
-      <update_rate>50</update_rate>
-      <num_wheel_pairs>2</num_wheel_pairs>
-      <left_joint>front_left_wheel_joint</left_joint>
-      <right_joint>front_right_wheel_joint</right_joint>
-      <left_joint>rear_left_wheel_joint</left_joint>
-      <right_joint>rear_right_wheel_joint</right_joint>
-      <wheel_separation>0.490</wheel_separation>
-      <wheel_separation>0.490</wheel_separation>
-      <wheel_diameter>0.180</wheel_diameter>
-      <wheel_diameter>0.180</wheel_diameter>
-      <max_wheel_torque>50.0</max_wheel_torque>
-      <max_wheel_acceleration>2.0</max_wheel_acceleration>
-      <publish_odom>true</publish_odom>
-      <publish_odom_tf>true</publish_odom_tf>
-      <publish_wheel_tf>true</publish_wheel_tf>
-      <odometry_frame>odom</odometry_frame>
-      <robot_base_frame>base_footprint</robot_base_frame>
-      <odometry_source>1</odometry_source>
-    </plugin>
-  </gazebo>
+  <xacro:macro name="scout_mini_gazebo" params="prefix:=''">
+    <!-- Material colors -->
+    <gazebo reference="${prefix}base_link">
+      <material>Gazebo/Yellow</material>
+    </gazebo>
+    <gazebo reference="${prefix}front_left_wheel_link">
+      <material>Gazebo/Black</material>
+      <mu1>1.0</mu1>
+      <mu2>1.0</mu2>
+      <kp>1000000.0</kp>
+      <kd>100.0</kd>
+    </gazebo>
+    <gazebo reference="${prefix}front_right_wheel_link">
+      <material>Gazebo/Black</material>
+      <mu1>1.0</mu1>
+      <mu2>1.0</mu2>
+      <kp>1000000.0</kp>
+      <kd>100.0</kd>
+    </gazebo>
+    <gazebo reference="${prefix}rear_left_wheel_link">
+      <material>Gazebo/Black</material>
+      <mu1>1.0</mu1>
+      <mu2>1.0</mu2>
+      <kp>1000000.0</kp>
+      <kd>100.0</kd>
+    </gazebo>
+    <gazebo reference="${prefix}rear_right_wheel_link">
+      <material>Gazebo/Black</material>
+      <mu1>1.0</mu1>
+      <mu2>1.0</mu2>
+      <kp>1000000.0</kp>
+      <kd>100.0</kd>
+    </gazebo>
+    <!-- ============================================================== -->
+    <!-- Skid-steer drive controller                                    -->
+    <!-- ============================================================== -->
+    <gazebo>
+      <plugin name="${prefix}skid_steer_controller" filename="libgazebo_ros_diff_drive.so">
+        <ros>
+          <namespace>/</namespace>
+          <remapping>cmd_vel:=cmd_vel</remapping>
+          <remapping>odom:=odom</remapping>
+        </ros>
+        <update_rate>50</update_rate>
+        <num_wheel_pairs>2</num_wheel_pairs>
+        <left_joint>${prefix}front_left_wheel_joint</left_joint>
+        <right_joint>${prefix}front_right_wheel_joint</right_joint>
+        <left_joint>${prefix}rear_left_wheel_joint</left_joint>
+        <right_joint>${prefix}rear_right_wheel_joint</right_joint>
+        <wheel_separation>0.490</wheel_separation>
+        <wheel_separation>0.490</wheel_separation>
+        <wheel_diameter>0.180</wheel_diameter>
+        <wheel_diameter>0.180</wheel_diameter>
+        <max_wheel_torque>50.0</max_wheel_torque>
+        <max_wheel_acceleration>2.0</max_wheel_acceleration>
+        <publish_odom>true</publish_odom>
+        <publish_odom_tf>true</publish_odom_tf>
+        <publish_wheel_tf>true</publish_wheel_tf>
+        <odometry_frame>${prefix}odom</odometry_frame>
+        <robot_base_frame>${prefix}base_footprint</robot_base_frame>
+        <odometry_source>1</odometry_source>
+      </plugin>
+    </gazebo>
+  </xacro:macro>
 </robot>

File: src/scout_mini_description/urdf/scout_mini.urdf.xacro (robot description, xacro)
@@ -14,5 +14,4 @@
   <xacro:property name="wheelbase"       value="0.452"/>
   <xacro:property name="track_width"     value="0.490"/>
-  <!-- Wheel vertical offset: bottom of base sits above ground by wheel_radius -->
   <xacro:property name="base_z_offset" value="${wheel_radius}"/>
   <!-- ============================================================== -->
@@ -38,39 +37,13 @@
   </xacro:macro>
   <!-- ============================================================== -->
-  <!-- base_footprint: virtual frame on the ground                    -->
+  <!-- Sensor modules                                                  -->
   <!-- ============================================================== -->
-  <link name="base_footprint"/>
-  <!-- ============================================================== -->
-  <!-- base_link: main body                                            -->
-  <!-- ============================================================== -->
-  <link name="base_link">
-    <visual>
-      <origin xyz="0 0 ${base_height/2}" rpy="0 0 0"/>
-      <geometry>
-        <box size="${base_length} ${base_width} ${base_height}"/>
-      </geometry>
-      <material name="scout_yellow">
-        <color rgba="0.95 0.75 0.05 1.0"/>
-      </material>
-    </visual>
-    <collision>
-      <origin xyz="0 0 ${base_height/2}" rpy="0 0 0"/>
-      <geometry>
-        <box size="${base_length} ${base_width} ${base_height}"/>
-      </geometry>
-    </collision>
-    <xacro:box_inertia m="${base_mass}" x="${base_length}" y="${base_width}" z="${base_height}"/>
-  </link>
-  <joint name="base_footprint_to_base_link" type="fixed">
-    <parent link="base_footprint"/>
-    <child link="base_link"/>
-    <origin xyz="0 0 ${base_z_offset}" rpy="0 0 0"/>
-  </joint>
+  <xacro:include filename="$(find scout_mini_description)/urdf/sensors/imu.xacro"/>
+  <xacro:include filename="$(find scout_mini_description)/urdf/sensors/lidar_2d.xacro"/>
   <!-- ============================================================== -->
   <!-- Wheel macro                                                     -->
-  <!-- Reused for all four wheels                                      -->
   <!-- ============================================================== -->
-  <xacro:macro name="wheel" params="prefix x_offset y_offset">
-    <link name="${prefix}_wheel_link">
+  <xacro:macro name="wheel" params="prefix wheel_name x_offset y_offset">
+    <link name="${prefix}${wheel_name}_wheel_link">
       <visual>
         <origin xyz="0 0 0" rpy="${pi/2} 0 0"/>
@@ -78,5 +51,5 @@
           <cylinder radius="${wheel_radius}" length="${wheel_width}"/>
         </geometry>
-        <material name="wheel_black">
+        <material name="wheel_black_${prefix}${wheel_name}">
           <color rgba="0.1 0.1 0.1 1.0"/>
         </material>
@@ -90,31 +63,80 @@
       <xacro:cylinder_inertia m="${wheel_mass}" r="${wheel_radius}" h="${wheel_width}"/>
     </link>
-    <joint name="${prefix}_wheel_joint" type="continuous">
-      <parent link="base_link"/>
-      <child link="${prefix}_wheel_link"/>
+    <joint name="${prefix}${wheel_name}_wheel_joint" type="continuous">
+      <parent link="${prefix}base_link"/>
+      <child link="${prefix}${wheel_name}_wheel_link"/>
       <origin xyz="${x_offset} ${y_offset} 0" rpy="0 0 0"/>
       <axis xyz="0 1 0"/>
     </joint>
   </xacro:macro>
-  <!-- Instantiate four wheels -->
-  <xacro:wheel prefix="front_left"  x_offset="${ wheelbase/2}" y_offset="${ track_width/2}"/>
-  <xacro:wheel prefix="front_right" x_offset="${ wheelbase/2}" y_offset="${-track_width/2}"/>
-  <xacro:wheel prefix="rear_left"   x_offset="${-wheelbase/2}" y_offset="${ track_width/2}"/>
-  <xacro:wheel prefix="rear_right"  x_offset="${-wheelbase/2}" y_offset="${-track_width/2}"/>
+  <!-- ============================================================== -->
+  <!-- Main robot macro                                                -->
+  <!-- ============================================================== -->
+  <xacro:macro name="scout_mini_robot" params="prefix:=''
+                                                use_imu:=true
+                                                use_lidar:=true
+                                                lidar_samples:=360
+                                                imu_rate:=100">
+    <!-- base_footprint -->
+    <link name="${prefix}base_footprint"/>
+    <!-- base_link -->
+    <link name="${prefix}base_link">
+      <visual>
+        <origin xyz="0 0 ${base_height/2}" rpy="0 0 0"/>
+        <geometry>
+          <box size="${base_length} ${base_width} ${base_height}"/>
+        </geometry>
+        <material name="scout_yellow_${prefix}">
+          <color rgba="0.95 0.75 0.05 1.0"/>
+        </material>
+      </visual>
+      <collision>
+        <origin xyz="0 0 ${base_height/2}" rpy="0 0 0"/>
+        <geometry>
+          <box size="${base_length} ${base_width} ${base_height}"/>
+        </geometry>
+      </collision>
+      <xacro:box_inertia m="${base_mass}" x="${base_length}" y="${base_width}" z="${base_height}"/>
+    </link>
+    <joint name="${prefix}base_footprint_to_base_link" type="fixed">
+      <parent link="${prefix}base_footprint"/>
+      <child link="${prefix}base_link"/>
+      <origin xyz="0 0 ${base_z_offset}" rpy="0 0 0"/>
+    </joint>
+    <!-- Four wheels -->
+    <xacro:wheel prefix="${prefix}" wheel_name="front_left"  x_offset="${ wheelbase/2}" y_offset="${ track_width/2}"/>
+    <xacro:wheel prefix="${prefix}" wheel_name="front_right" x_offset="${ wheelbase/2}" y_offset="${-track_width/2}"/>
+    <xacro:wheel prefix="${prefix}" wheel_name="rear_left"   x_offset="${-wheelbase/2}" y_offset="${ track_width/2}"/>
+    <xacro:wheel prefix="${prefix}" wheel_name="rear_right"  x_offset="${-wheelbase/2}" y_offset="${-track_width/2}"/>
+    <!-- Conditional sensors -->
+    <xacro:if value="${use_imu}">
+      <xacro:imu_sensor
+        name="${prefix}imu"
+        parent="${prefix}base_link"
+        xyz="0 0 ${base_height + 0.01}"
+        rpy="0 0 0"
+        rate="${imu_rate}"
+        topic="imu"/>
+    </xacro:if>
+    <xacro:if value="${use_lidar}">
+      <xacro:lidar_2d_sensor
+        name="${prefix}lidar"
+        parent="${prefix}base_link"
+        xyz="0.20 0 ${base_height + 0.03}"
+        rpy="0 0 0"
+        samples="${lidar_samples}"
+        topic="scan"/>
+    </xacro:if>
+    <!-- Gazebo (per-instance: material + plugins) -->
+    <xacro:scout_mini_gazebo prefix="${prefix}"/>
+  </xacro:macro>
+  <!-- ============================================================== -->
+  <!-- Include the Gazebo macro definition                             -->
+  <!-- ============================================================== -->
   <xacro:include filename="$(find scout_mini_description)/urdf/scout_mini.gazebo.xacro"/>
   <!-- ============================================================== -->
-  <!-- Sensor modules                                                  -->
+  <!-- Instantiate one robot with empty prefix (Scene 1 compatibility) -->
+  <!-- This is overridden when launched via spawn_robot.launch.py      -->
   <!-- ============================================================== -->
-  <xacro:include filename="$(find scout_mini_description)/urdf/sensors/imu.xacro"/>
-  <xacro:include filename="$(find scout_mini_description)/urdf/sensors/lidar_2d.xacro"/>
-  <xacro:imu_sensor
-    name="imu"
-    parent="base_link"
-    xyz="0 0 ${base_height + 0.01}"
-    rpy="0 0 0"/>
-  <xacro:lidar_2d_sensor
-    name="lidar"
-    parent="base_link"
-    xyz="0.20 0 ${base_height + 0.03}"
-    rpy="0 0 0"/>
+  <xacro:scout_mini_robot prefix=""/>
 </robot>
