Commit message: Multi-robot support via ROS2 namespaces; heterogeneous fleet of 3

File: src/scout_mini_description/urdf/scout_mini.gazebo.xacro (robot description, xacro)
@@ -1,13 +1,9 @@
 <?xml version="1.0"?>
 <robot xmlns:xacro="http://www.ros.org/wiki/xacro">
-  <!-- ============================================================== -->
-  <!-- Gazebo macro: per-robot material + skid-steer plugin            -->
-  <!-- ============================================================== -->
-  <xacro:macro name="scout_mini_gazebo" params="prefix:=''">
-    <!-- Material colors -->
-    <gazebo reference="${prefix}base_link">
+  <xacro:macro name="scout_mini_gazebo" params="namespace:=''">
+    <gazebo reference="base_link">
       <material>Gazebo/Yellow</material>
     </gazebo>
-    <gazebo reference="${prefix}front_left_wheel_link">
+    <gazebo reference="front_left_wheel_link">
       <material>Gazebo/Black</material>
       <mu1>1.0</mu1>
@@ -16,5 +12,5 @@
       <kd>100.0</kd>
     </gazebo>
-    <gazebo reference="${prefix}front_right_wheel_link">
+    <gazebo reference="front_right_wheel_link">
       <material>Gazebo/Black</material>
       <mu1>1.0</mu1>
@@ -23,5 +19,5 @@
       <kd>100.0</kd>
     </gazebo>
-    <gazebo reference="${prefix}rear_left_wheel_link">
+    <gazebo reference="rear_left_wheel_link">
       <material>Gazebo/Black</material>
       <mu1>1.0</mu1>
@@ -30,5 +26,5 @@
       <kd>100.0</kd>
     </gazebo>
-    <gazebo reference="${prefix}rear_right_wheel_link">
+    <gazebo reference="rear_right_wheel_link">
       <material>Gazebo/Black</material>
       <mu1>1.0</mu1>
@@ -37,11 +33,8 @@
       <kd>100.0</kd>
     </gazebo>
-    <!-- ============================================================== -->
-    <!-- Skid-steer drive controller                                    -->
-    <!-- ============================================================== -->
     <gazebo>
-      <plugin name="${prefix}skid_steer_controller" filename="libgazebo_ros_diff_drive.so">
+      <plugin name="skid_steer_controller" filename="libgazebo_ros_diff_drive.so">
         <ros>
-          <namespace>/</namespace>
+          <namespace>${namespace}</namespace>
           <remapping>cmd_vel:=cmd_vel</remapping>
           <remapping>odom:=odom</remapping>
@@ -49,8 +42,8 @@
         <update_rate>50</update_rate>
         <num_wheel_pairs>2</num_wheel_pairs>
-        <left_joint>${prefix}front_left_wheel_joint</left_joint>
-        <right_joint>${prefix}front_right_wheel_joint</right_joint>
-        <left_joint>${prefix}rear_left_wheel_joint</left_joint>
-        <right_joint>${prefix}rear_right_wheel_joint</right_joint>
+        <left_joint>front_left_wheel_joint</left_joint>
+        <right_joint>front_right_wheel_joint</right_joint>
+        <left_joint>rear_left_wheel_joint</left_joint>
+        <right_joint>rear_right_wheel_joint</right_joint>
         <wheel_separation>0.490</wheel_separation>
         <wheel_separation>0.490</wheel_separation>
@@ -62,6 +55,6 @@
         <publish_odom_tf>true</publish_odom_tf>
         <publish_wheel_tf>true</publish_wheel_tf>
-        <odometry_frame>${prefix}odom</odometry_frame>
-        <robot_base_frame>${prefix}base_footprint</robot_base_frame>
+        <odometry_frame>odom</odometry_frame>
+        <robot_base_frame>base_footprint</robot_base_frame>
         <odometry_source>1</odometry_source>
       </plugin>

File: src/scout_mini_description/urdf/scout_mini.urdf.xacro (robot description, xacro)
@@ -3,5 +3,4 @@
   <!-- ============================================================== -->
   <!-- Properties: Scout Mini physical parameters                     -->
-  <!-- Source: AgileX official specifications                          -->
   <!-- ============================================================== -->
   <xacro:property name="base_length" value="0.612"/>
@@ -15,4 +14,10 @@
   <xacro:property name="track_width"     value="0.490"/>
   <xacro:property name="base_z_offset" value="${wheel_radius}"/>
+  <!-- Launch-supplied arguments -->
+  <xacro:arg name="namespace" default=""/>
+  <xacro:arg name="use_imu" default="true"/>
+  <xacro:arg name="use_lidar" default="true"/>
+  <xacro:arg name="lidar_samples" default="360"/>
+  <xacro:arg name="imu_rate" default="100"/>
   <!-- ============================================================== -->
   <!-- Inertial macros                                                 -->
@@ -37,13 +42,44 @@
   </xacro:macro>
   <!-- ============================================================== -->
-  <!-- Sensor modules                                                  -->
+  <!-- Sensor and gazebo includes                                      -->
   <!-- ============================================================== -->
   <xacro:include filename="$(find scout_mini_description)/urdf/sensors/imu.xacro"/>
   <xacro:include filename="$(find scout_mini_description)/urdf/sensors/lidar_2d.xacro"/>
+  <xacro:include filename="$(find scout_mini_description)/urdf/scout_mini.gazebo.xacro"/>
+  <!-- ============================================================== -->
+  <!-- base_footprint                                                  -->
+  <!-- ============================================================== -->
+  <link name="base_footprint"/>
+  <!-- ============================================================== -->
+  <!-- base_link                                                       -->
+  <!-- ============================================================== -->
+  <link name="base_link">
+    <visual>
+      <origin xyz="0 0 ${base_height/2}" rpy="0 0 0"/>
+      <geometry>
+        <box size="${base_length} ${base_width} ${base_height}"/>
+      </geometry>
+      <material name="scout_yellow">
+        <color rgba="0.95 0.75 0.05 1.0"/>
+      </material>
+    </visual>
+    <collision>
+      <origin xyz="0 0 ${base_height/2}" rpy="0 0 0"/>
+      <geometry>
+        <box size="${base_length} ${base_width} ${base_height}"/>
+      </geometry>
+    </collision>
+    <xacro:box_inertia m="${base_mass}" x="${base_length}" y="${base_width}" z="${base_height}"/>
+  </link>
+  <joint name="base_footprint_to_base_link" type="fixed">
+    <parent link="base_footprint"/>
+    <child link="base_link"/>
+    <origin xyz="0 0 ${base_z_offset}" rpy="0 0 0"/>
+  </joint>
   <!-- ============================================================== -->
   <!-- Wheel macro                                                     -->
   <!-- ============================================================== -->
-  <xacro:macro name="wheel" params="prefix wheel_name x_offset y_offset">
-    <link name="${prefix}${wheel_name}_wheel_link">
+  <xacro:macro name="wheel" params="prefix x_offset y_offset">
+    <link name="${prefix}_wheel_link">
       <visual>
         <origin xyz="0 0 0" rpy="${pi/2} 0 0"/>
@@ -51,5 +87,5 @@
           <cylinder radius="${wheel_radius}" length="${wheel_width}"/>
         </geometry>
-        <material name="wheel_black_${prefix}${wheel_name}">
+        <material name="wheel_black">
           <color rgba="0.1 0.1 0.1 1.0"/>
         </material>
@@ -63,80 +99,40 @@
       <xacro:cylinder_inertia m="${wheel_mass}" r="${wheel_radius}" h="${wheel_width}"/>
     </link>
-    <joint name="${prefix}${wheel_name}_wheel_joint" type="continuous">
-      <parent link="${prefix}base_link"/>
-      <child link="${prefix}${wheel_name}_wheel_link"/>
+    <joint name="${prefix}_wheel_joint" type="continuous">
+      <parent link="base_link"/>
+      <child link="${prefix}_wheel_link"/>
       <origin xyz="${x_offset} ${y_offset} 0" rpy="0 0 0"/>
       <axis xyz="0 1 0"/>
     </joint>
   </xacro:macro>
+  <!-- Instantiate four wheels -->
+  <xacro:wheel prefix="front_left"  x_offset="${ wheelbase/2}" y_offset="${ track_width/2}"/>
+  <xacro:wheel prefix="front_right" x_offset="${ wheelbase/2}" y_offset="${-track_width/2}"/>
+  <xacro:wheel prefix="rear_left"   x_offset="${-wheelbase/2}" y_offset="${ track_width/2}"/>
+  <xacro:wheel prefix="rear_right"  x_offset="${-wheelbase/2}" y_offset="${-track_width/2}"/>
   <!-- ============================================================== -->
-  <!-- Main robot macro                                                -->
+  <!-- Conditional sensors                                             -->
   <!-- ============================================================== -->
-  <xacro:macro name="scout_mini_robot" params="prefix:=''
-                                                use_imu:=true
-                                                use_lidar:=true
-                                                lidar_samples:=360
-                                                imu_rate:=100">
-    <!-- base_footprint -->
-    <link name="${prefix}base_footprint"/>
-    <!-- base_link -->
-    <link name="${prefix}base_link">
-      <visual>
-        <origin xyz="0 0 ${base_height/2}" rpy="0 0 0"/>
-        <geometry>
-          <box size="${base_length} ${base_width} ${base_height}"/>
-        </geometry>
-        <material name="scout_yellow_${prefix}">
-          <color rgba="0.95 0.75 0.05 1.0"/>
-        </material>
-      </visual>
-      <collision>
-        <origin xyz="0 0 ${base_height/2}" rpy="0 0 0"/>
-        <geometry>
-          <box size="${base_length} ${base_width} ${base_height}"/>
-        </geometry>
-      </collision>
-      <xacro:box_inertia m="${base_mass}" x="${base_length}" y="${base_width}" z="${base_height}"/>
-    </link>
-    <joint name="${prefix}base_footprint_to_base_link" type="fixed">
-      <parent link="${prefix}base_footprint"/>
-      <child link="${prefix}base_link"/>
-      <origin xyz="0 0 ${base_z_offset}" rpy="0 0 0"/>
-    </joint>
-    <!-- Four wheels -->
-    <xacro:wheel prefix="${prefix}" wheel_name="front_left"  x_offset="${ wheelbase/2}" y_offset="${ track_width/2}"/>
-    <xacro:wheel prefix="${prefix}" wheel_name="front_right" x_offset="${ wheelbase/2}" y_offset="${-track_width/2}"/>
-    <xacro:wheel prefix="${prefix}" wheel_name="rear_left"   x_offset="${-wheelbase/2}" y_offset="${ track_width/2}"/>
-    <xacro:wheel prefix="${prefix}" wheel_name="rear_right"  x_offset="${-wheelbase/2}" y_offset="${-track_width/2}"/>
-    <!-- Conditional sensors -->
-    <xacro:if value="${use_imu}">
-      <xacro:imu_sensor
-        name="${prefix}imu"
-        parent="${prefix}base_link"
-        xyz="0 0 ${base_height + 0.01}"
-        rpy="0 0 0"
-        rate="${imu_rate}"
-        topic="imu"/>
-    </xacro:if>
-    <xacro:if value="${use_lidar}">
-      <xacro:lidar_2d_sensor
-        name="${prefix}lidar"
-        parent="${prefix}base_link"
-        xyz="0.20 0 ${base_height + 0.03}"
-        rpy="0 0 0"
-        samples="${lidar_samples}"
-        topic="scan"/>
-    </xacro:if>
-    <!-- Gazebo (per-instance: material + plugins) -->
-    <xacro:scout_mini_gazebo prefix="${prefix}"/>
-  </xacro:macro>
-  <!-- ============================================================== -->
-  <!-- Include the Gazebo macro definition                             -->
-  <!-- ============================================================== -->
-  <xacro:include filename="$(find scout_mini_description)/urdf/scout_mini.gazebo.xacro"/>
-  <!-- ============================================================== -->
-  <!-- Instantiate one robot with empty prefix (Scene 1 compatibility) -->
-  <!-- This is overridden when launched via spawn_robot.launch.py      -->
-  <!-- ============================================================== -->
-  <xacro:scout_mini_robot prefix=""/>
+  <xacro:if value="$(arg use_imu)">
+    <xacro:imu_sensor
+      name="imu"
+      parent="base_link"
+      xyz="0 0 ${base_height + 0.01}"
+      rpy="0 0 0"
+      rate="$(arg imu_rate)"
+      namespace="$(arg namespace)"
+      topic="imu"/>
+  </xacro:if>
+  <xacro:if value="$(arg use_lidar)">
+    <xacro:lidar_2d_sensor
+      name="lidar"
+      parent="base_link"
+      xyz="0.20 0 ${base_height + 0.03}"
+      rpy="0 0 0"
+      samples="$(arg lidar_samples)"
+      namespace="$(arg namespace)"
+      topic="scan"/>
+  </xacro:if>
+  <!-- Gazebo material + skid-steer plugin -->
+  <xacro:scout_mini_gazebo namespace="$(arg namespace)"/>
 </robot>

File: src/scout_mini_description/urdf/sensors/imu.xacro (robot description, xacro)
@@ -1,25 +1,10 @@
 <?xml version="1.0"?>
 <robot xmlns:xacro="http://www.ros.org/wiki/xacro">
-  <!-- ============================================================== -->
-  <!-- IMU sensor module                                               -->
-  <!--                                                                 -->
-  <!-- Self-contained: link, joint, Gazebo plugin in one macro.        -->
-  <!--                                                                 -->
-  <!-- Parameters:                                                     -->
-  <!--   name          : unique name for this sensor instance         -->
-  <!--   parent        : link to attach to                             -->
-  <!--   xyz           : mount position relative to parent             -->
-  <!--   rpy           : mount orientation relative to parent          -->
-  <!--   rate          : publish rate in Hz (default 100)              -->
-  <!--   gyro_stddev   : gyroscope noise std dev (default 2e-4)        -->
-  <!--   accel_stddev  : accelerometer noise std dev (default 1.7e-2)  -->
-  <!--   topic         : output topic name (default /imu)              -->
-  <!-- ============================================================== -->
   <xacro:macro name="imu_sensor" params="name parent xyz rpy
                                           rate:=100
                                           gyro_stddev:=0.0002
                                           accel_stddev:=0.017
-                                          topic:=imu">
-    <!-- Physical link -->
+                                          topic:=imu
+                                          namespace:=''">
     <link name="${name}_link">
       <visual>
@@ -49,5 +34,4 @@
       <origin xyz="${xyz}" rpy="${rpy}"/>
     </joint>
-    <!-- Gazebo IMU plugin -->
     <gazebo reference="${name}_link">
       <sensor name="${name}_sensor" type="imu">
@@ -58,5 +42,5 @@
         <plugin filename="libgazebo_ros_imu_sensor.so" name="${name}_plugin">
           <ros>
-            <namespace>/</namespace>
+            <namespace>${namespace}</namespace>
             <remapping>~/out:=${topic}</remapping>
           </ros>

File: src/scout_mini_description/urdf/sensors/lidar_2d.xacro (robot description, xacro)
@@ -1,22 +1,4 @@
 <?xml version="1.0"?>
 <robot xmlns:xacro="http://www.ros.org/wiki/xacro">
-  <!-- ============================================================== -->
-  <!-- 2D Lidar sensor module                                          -->
-  <!--                                                                 -->
-  <!-- Self-contained: link, joint, Gazebo plugin in one macro.        -->
-  <!--                                                                 -->
-  <!-- Parameters:                                                     -->
-  <!--   name           : unique name for this sensor instance        -->
-  <!--   parent         : link to attach to                            -->
-  <!--   xyz            : mount position relative to parent            -->
-  <!--   rpy            : mount orientation relative to parent         -->
-  <!--   samples        : angular samples per scan (default 360)       -->
-  <!--   update_rate    : scan rate in Hz (default 10)                 -->
-  <!--   min_range      : minimum range in m (default 0.12)            -->
-  <!--   max_range      : maximum range in m (default 12.0)            -->
-  <!--   noise_stddev   : range noise std dev (default 0.01)           -->
-  <!--   topic          : output topic name (default /scan)            -->
-  <!--   visualize      : show rays in Gazebo (default true)           -->
-  <!-- ============================================================== -->
   <xacro:macro name="lidar_2d_sensor" params="name parent xyz rpy
                                                samples:=360
@@ -26,6 +8,6 @@
                                                noise_stddev:=0.01
                                                topic:=scan
+                                               namespace:=''
                                                visualize:=true">
-    <!-- Physical link -->
     <link name="${name}_link">
       <visual>
@@ -55,5 +37,4 @@
       <origin xyz="${xyz}" rpy="${rpy}"/>
     </joint>
-    <!-- Gazebo 2D Lidar plugin -->
     <gazebo reference="${name}_link">
       <sensor name="${name}_sensor" type="ray">
@@ -84,5 +65,5 @@
         <plugin filename="libgazebo_ros_ray_sensor.so" name="${name}_plugin">
           <ros>
-            <namespace>/</namespace>
+            <namespace>${namespace}</namespace>
             <remapping>~/out:=${topic}</remapping>
           </ros>
